File: hardware/pmod/kicad/pmod_1553.sch (KiCad schematic (older format))
At the start: 35 parts, among them IC1 TB001-500-02BE, IC2 TB001-500-02BE, J1 Conn_02x06_Top_Bottom, J2 Conn_01x02, J3 Conn_01x02, P1 78604-9JC, P2 78604-9JC, U1 74HC14, U2 VO2630, U3 VO2630

Commit message: added bill of materials
Parts:
- C1: Vendor (none) -> https://www.mouser.com/ProductDetail/647-UPW1A220MDD
- C2: Vendor (none) -> https://www.mouser.com/ProductDetail/TDK/CK45-B3AD102KYNNA?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
- C3, C4: Vendor (none) -> https://www.mouser.com/ProductDetail/TDK/FK18C0G1H100D?qs=k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
- C5: Vendor (none) -> https://www.mouser.com/ProductDetail/TDK/FK26C0G1H104J?qs=z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
- C6, C9: Vendor (none) -> https://www.mouser.com/ProductDetail/TDK/FK18C0G1H220J?qs=k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
- IC1, IC2: Vendor (none) -> https://www.mouser.com/ProductDetail/CUI-Devices/TB001-500-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
- J1: Vendor (none) -> https://www.mouser.com/ProductDetail/Amphenol-FCI/10129382-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
- J2, J3: Vendor (none) -> https://www.mouser.com/ProductDetail/Molex/22-29-2021?qs=5g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
- P1, P2: Vendor (none) -> https://www.mouser.com/ProductDetail/Murata-Power-Solutions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
- PS1: Vendor (none) -> https://www.mouser.com/ProductDetail/TRACO-Power/TBA-1-0311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
- R1, R11, R12, R2, R3, R4, R5, R6, R7, R8: Vendor (none) -> https://www.mouser.com/ProductDetail/TE-Connectivity-Holswo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
- R10, R9: value 330_2K2-DNP -> 332_2K2-DNP; Vendor (none) -> https://www.mouser.com/ProductDetail/TE-Connectivity-Holswo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
- U1: Vendor (none) -> https://www.mouser.com/ProductDetail/Texas-Instruments/SN74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
- U1: footprint (none) -> Package_DIP:DIP-14_W7.62mm_LongPads
- U2, U3: Vendor (none) -> https://www.mouser.com/ProductDetail/Vishay-Semiconductors/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

Commit message: kicad url updates, they break removing the ? and after, but its clearer in seeing the make/model
Parts:
- C2: Vendor https://www.mouser.com/ProductDetail/TDK/CK45-B3AD102KYNNA?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 -> https://www.mouser.com/ProductDetail/TDK/CK45-B3AD102KYNNA
- C3, C4: Vendor https://www.mouser.com/ProductDetail/TDK/FK18C0G1H100D?qs=k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 -> https://www.mouser.com/ProductDetail/TDK/FK18C0G1H100D
- C5: Vendor https://www.mouser.com/ProductDetail/TDK/FK26C0G1H104J?qs=z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 -> https://www.mouser.com/ProductDetail/TDK/FK26C0G1H104J
- C6, C9: Vendor https://www.mouser.com/ProductDetail/TDK/FK18C0G1H220J?qs=k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 -> https://www.mouser.com/ProductDetail/TDK/FK18C0G1H220J
- C7, C8: Vendor (none) -> https://www.mouser.com/ProductDetail/TDK/FK26C0G1H104J
- IC1, IC2: Vendor https://www.mouser.com/ProductDetail/CUI-Devices/TB001-500-02BE?qs=%2Fha2pyFadujMdv6PiXeNZkSsm5Qkxr1FY4D5p2i4LtbuG6HS8Lj7%2Fg%3D%3D -> https://www.mouser.com/ProductDetail/CUI-Devices/TB001-500-02BE
- J1: Vendor https://www.mouser.com/ProductDetail/Amphenol-FCI/10129382-912001BLF?qs=%2Fha2pyFadug32m4xOB2%252BmVXU3aKMd9PcTrSHZ%252BY316jfSjjQJuKTrO0vID2tiybT -> https://www.mouser.com/ProductDetail/Amphenol-FCI/10129382-912001BLF
- J2, J3: Vendor https://www.mouser.com/ProductDetail/Molex/22-29-2021?qs=5g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 -> https://www.mouser.com/ProductDetail/Molex/22-29-2021
- P2: Vendor https://www.mouser.com/ProductDetail/Murata-Power-Solutions/78604-9JC?qs=f4NXQ36d%252BdAJuzG35nIgNw%3D%3D -> https://www.mouser.com/ProductDetail/Murata-Power-Solutions/78604-9JC
- PS1: Vendor https://www.mouser.com/ProductDetail/TRACO-Power/TBA-1-0311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 -> https://www.mouser.com/ProductDetail/TRACO-Power/TBA-1-0311
- R1, R11, R12, R2, R3, R4: Vendor https://www.mouser.com/ProductDetail/TE-Connectivity-Holsworthy/YR1B100RCC?qs=%2Fha2pyFadujfkjl%2Fw2CT8wH4dU44PFFTyZyFDkshbTA0fGbLwSa2EA%3D%3D -> https://www.mouser.com/ProductDetail/TE-Connectivity-Holsworthy/YR1B100RCC
- R10, R9: Vendor https://www.mouser.com/ProductDetail/TE-Connectivity-Holsworthy/YR1B332RCC?qs=%2Fha2pyFadug6BvjU2YViCydgO3v3mIlvjAYlexUPMTr57zwxvr%252B3rg%3D%3D -> https://www.mouser.com/ProductDetail/TE-Connectivity-Holsworthy/YR1B332RCC
- R7, R8: Vendor https://www.mouser.com/ProductDetail/TE-Connectivity-Holsworthy/YR1B49R9CC?qs=%2Fha2pyFaduj9DVYKP1mQ5I6cbHeSbqcRTxxAPrgoG9nIERwP%252BGOgJQ%3D%3D -> https://www.mouser.com/ProductDetail/TE-Connectivity-Holsworthy/YR1B49R9CC
- U1: Vendor https://www.mouser.com/ProductDetail/Texas-Instruments/SN74HC14AN?qs=byeeYqUIh0NMy3GLE70Pnw%3D%3D -> https://www.mouser.com/ProductDetail/Texas-Instruments/SN74HC14AN
- U3: Vendor https://www.mouser.com/ProductDetail/Vishay-Semiconductors/VO2630?qs=xCMk%252BIHWTZOuc1EdsOwr1g%3D%3D -> https://www.mouser.com/ProductDetail/Vishay-Semiconductors/VO2630

Commit message: bom updates
Parts:
- C1: Vendor https://www.mouser.com/ProductDetail/647-UPW1A220MDD -> Nichicon/647-UPW1A220MDD
- C2: Vendor https://www.mouser.com/ProductDetail/TDK/CK45-B3AD102KYNNA -> TDK/CK45-B3AD102KYNNA
- C3, C4: Vendor https://www.mouser.com/ProductDetail/TDK/FK18C0G1H100D -> TDK/FK18C0G1H100D
- C5, C7, C8: Vendor https://www.mouser.com/ProductDetail/TDK/FK26C0G1H104J -> TDK/FK26C0G1H104J
- C6, C9: Vendor https://www.mouser.com/ProductDetail/TDK/FK18C0G1H220J -> TDK/FK18C0G1H220J
- IC1, IC2: Vendor https://www.mouser.com/ProductDetail/CUI-Devices/TB001-500-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 -> CUI-Devices/TB001-500-02BE
- J1: Vendor https://www.mouser.com/ProductDetail/Amphenol-FCI/10129382-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 -> Amphenol-FCI/10129382-912001BLF
- J2, J3: Vendor https://www.mouser.com/ProductDetail/Molex/22-29-2021 -> Molex/22-29-2021
- P1, P2: Vendor https://www.mouser.com/ProductDetail/Murata-Power-Solutions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 -> Murata-Power-Solutions/78604-9JC
- PS1: Vendor https://www.mouser.com/ProductDetail/TRACO-Power/TBA-1-0311 -> TRACO-Power/TBA-1-0311
- R1, R11, R12, R2, R3, R4: Vendor https://www.mouser.com/ProductDetail/TE-Connectivity-Holswo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 -> TE-Connectivity-Holsworthy/YR1B100RCC
- R10, R9: Vendor https://www.mouser.com/ProductDetail/TE-Connectivity-Holswo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 -> TE-Connectivity-Holsworthy/YR1B332RCC
- R5, R6: Vendor https://www.mouser.com/ProductDetail/TE-Connectivity-Holswo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 -> TE-Connectivity-Holsworthy/YR1B49R9CC?qs=%2Fha2pyFaduj9DVYK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
- R7, R8: Vendor https://www.mouser.com/ProductDetail/TE-Connectivity-Holswo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 -> TE-Connectivity-Holsworthy/YR1B49R9CC
- U1: Vendor https://www.mouser.com/ProductDetail/Texas-Instruments/SN74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 -> Texas-Instruments/SN74HC14AN
- U2: Vendor https://www.mouser.com/ProductDetail/Vishay-Semiconductors/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 -> Vishay-Semiconductors/VO2630?qs=xCMk%252BIHWTZOuc1EdsOwr1g%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
- U3: Vendor https://www.mouser.com/ProductDetail/Vishay-Semiconductors/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 -> Vishay-Semiconductors/VO2630

Commit message: added adg413 switch to pmod1553, added symbols and data sheets for the adg413 and mcp6d11.
Parts:
- removed C6, C9: 22pF_DNP, Capacitor_THT:C_Disc_D4.7mm_W2.5mm_P5.00mm, symbol Device:C
- removed IC1: TB001-500-02BE, cui:TB00150002BE, symbol TB001-500-02BE:TB001-500-02BE
- removed P1: 78604-9JC, murata_pulse_transformers:78604-9JC, symbol Murata_Pulse_Transformers:78604-9JC
- removed R5, R6: 49R9, Resistor_THT:R_Axial_DIN0207_L6.3mm_D2.5mm_P7.62mm_Horizontal, symbol Device:R
- added C10: 100NF, Capacitor_THT:C_Disc_D4.7mm_W2.5mm_P5.00mm, symbol Device:C
- added IC1: ADG413BNZ, Package_DIP:DIP-16_W7.62mm_LongPads, symbol ADG413BNZ:ADG413BNZ
Connections:
- net GNDD: now also C10.2, IC1.4 (VSS), IC1.5 (GND); no longer U1.5
- net at J1.12 (Pin_12): now also U1.5
- net at C4.1, R12.2, U2.6 (VO2): now also IC1.15 (D2)
- net at C3.2, R11.1, U2.7 (VO1): now also IC1.10 (D3)
- net at C7.2, C8.1, PS1.5 (+VOUT)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: now also C10.1, IC1.12 (VL), IC1.13 (VDD)
- net at R3.1: now also IC1.2 (D1); no longer P2.4
- net at R4.1: now also IC1.7 (D4); no longer P2.6
- net at U1.6: now also IC1.1 (IN1), IC1.16 (IN2), IC1.8 (IN4), IC1.9 (IN3)
- new net: IC1.11 (S3), IC1.6 (S4), P2.4
- new net: IC1.14 (S2), IC1.3 (S1), P2.6
Other:
- moved on the sheet: C1, C2, C3, C4, C5, C7, C8, H1, H2, IC2, J1, J2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
